File: kicad-eboard/kicad-eboard.sch (KiCad schematic (older format))
At the start: 7 parts

Commit message: Add TinkerBoard symbol
Parts:
- added BT?: Battery, symbol Device:Battery
- added U?: TinkerBoard, symbol 2019Spacehawks:TinkerBoard
Connections:
- wire segments 18 -> 20
Changed lines of the file:
@@
 $EndComp
 Wire Wire Line
-	1450 5700 2050 5700
+	1450 5700 1950 5700
 Wire Wire Line
 	2650 5700 2900 5700
@@
 	2900 5950 2900 6100
 Wire Wire Line
-	2900 6100 1450 6100
+	2900 6100 1950 6100
 $Comp
 L Relay_SolidState:34.81-8240 U?
@@
 F8 "GND" I L 2350 2900 50
 $EndSheet
+$Comp
+L Device:Battery BT?
+U 1 1 5D9D77E5
+P 1950 5900
+F 0 "BT?" H 2058 5946 50  0000 L CNN
+F 1 "Battery" H 2058 5855 50  0000 L CNN
+F 2 "" V 1950 5960 50  0001 C CNN
+F 3 "~" V 1950 5960 50  0001 C CNN
+	1    1950 5900
+	1    0    0    -1
+$EndComp
+Connection ~ 1950 5700
+Wire Wire Line
+	1950 5700 2050 5700
+Connection ~ 1950 6100
+Wire Wire Line
+	1950 6100 1450 6100
+$Comp
+L 2019Spacehawks:TinkerBoard U?
+U 1 1 5D9DC73D
+P 6000 2100
+F 0 "U?" H 5122 1496 50  0000 R CNN
+F 1 "TinkerBoard" H 5122 1405 50  0000 R CNN
+F 2 "" H 6000 2100 50  0001 C CNN
+F 3 "" H 6000 2100 50  0001 C CNN
+	1    6000 2100
+	1    0    0    -1
+$EndComp
 $EndSCHEMATC

Commit message: Add DC-DC converters
Parts:
- added U?: PDQ15-Q24-S12-D, symbol 2019Spacehawks:PDQXX-D_DC-DC_converter
- added U?: PDQ30-Q24-S5-D, symbol 2019Spacehawks:PDQXX-D_DC-DC_converter
Connections:
- net labels added: +12V, +5V, +BATT, GNDA, GNDPWR
- wire segments 20 -> 28
Other:
- moved on the sheet: BT?, CB?, SW?, U?

Commit message: Fill in some power topology
Parts:
- added C? (x2): 0.1u, symbol Device:C_Small
- added M? (x4): Motor_DC, symbol Motor:Motor_DC
- added R? (x2): 10K, symbol Device:R
- added U? (x2): Sabertooth2x60, symbol 2019Spacehawks:Sabertooth2x60
Connections:
- net labels added: GNDD, PWM0, PWM1
- wire segments 28 -> 82
- no-connect marks 0 -> 6

Commit message: Satisfy some ERC things
Parts:
- gave numbers to parts that had none: 21
Connections:
- net labels added: PWM[0..15]
- wire segments 82 -> 83
- no-connect marks 6 -> 4

Commit message: Add input filtering, trim to DC-DCs
Parts:
- added C? (x2): 100u, symbol Device:CP
- added C? (x2): 1u, symbol Device:C
- added C? (x2): 10n, symbol Device:C
- added L? (x2): 15u, symbol Device:L
- added MES?: Voltmeter_DC, symbol Device:Voltmeter_DC
- added RV? (x2): 10K, symbol Device:R_POT
- SW1: value SW_SPST -> ESTOP
- SW2: value SW_SPST -> REMOTE
- SW3: value SW_SPST -> POWER
Connections:
- wire segments 83 -> 107

Commit message: Add TinkerBoard decoupling caps
Parts:
- added C?: 1u, symbol Device:C
- added C?: 10n, symbol Device:C
Connections:
- wire segments 107 -> 113
Changed lines of the file:
@@
 	7900 2300 8400 2300
 Connection ~ 8400 2300
+$Comp
+L power:+5V #PWR?
+U 1 1 5DAAA77D
+P 1300 2550
+F 0 "#PWR?" H 1300 2400 50  0001 C CNN
+F 1 "+5V" H 1300 2690 50  0000 C CNN
+F 2 "" H 1300 2550 50  0001 C CNN
+F 3 "" H 1300 2550 50  0001 C CNN
+	1    1300 2550
+	1    0    0    -1
+$EndComp
+$Comp
+L power:GNDD #PWR?
+U 1 1 5DAAA808
+P 1300 2950
+F 0 "#PWR?" H 1300 2700 50  0001 C CNN
+F 1 "GNDD" H 1300 2825 50  0000 C CNN
+F 2 "" H 1300 2950 50  0001 C CNN
+F 3 "" H 1300 2950 50  0001 C CNN
+	1    1300 2950
+	1    0    0    -1
+$EndComp
+$Comp
+L Device:C C?
+U 1 1 5DAAAF8B
+P 1150 2750
+F 0 "C?" H 1175 2850 50  0000 L CNN
+F 1 "1u" H 1175 2650 50  0000 L CNN
+F 2 "" H 1188 2600 50  0001 C CNN
+F 3 "~" H 1150 2750 50  0001 C CNN
+	1    1150 2750
+	1    0    0    -1
+$EndComp
+$Comp
+L Device:C C?
+U 1 1 5DAAAF91
+P 1450 2750
+F 0 "C?" H 1475 2850 50  0000 L CNN
+F 1 "10n" H 1475 2650 50  0000 L CNN
+F 2 "" H 1488 2600 50  0001 C CNN
+F 3 "~" H 1450 2750 50  0001 C CNN
+	1    1450 2750
+	1    0    0    -1
+$EndComp
+Wire Wire Line
+	1150 2600 1300 2600
+Wire Wire Line
+	1150 2900 1300 2900
+Wire Wire Line
+	1300 2950 1300 2900
+Connection ~ 1300 2900
+Wire Wire Line
+	1300 2900 1450 2900
+Wire Wire Line
+	1300 2600 1300 2550
+Connection ~ 1300 2600
+Wire Wire Line
+	1300 2600 1450 2600
 Wire Bus Line
 	5600 2400 5600 4850

Commit message: Update SSR
Parts:
- U3: value 34.81-8240 -> DC100D100CH; footprint OptoDevice:Finder_34.81 -> (none)
Changed lines of the file:
@@
 P 5350 1350
 F 0 "U3" H 5350 1675 50  0000 C CNN
-F 1 "34.81-8240" H 5350 1584 50  0000 C CNN
-F 2 "OptoDevice:Finder_34.81" H 5150 1150 50  0001 L CIN
-F 3 "https://gfinder.findernet.com/public/attachments/34/EN/S34USAEN.pdf" H 5325 1350 50  0001 L CNN
+F 1 "DC100D100CH" H 5350 1584 50  0000 C CNN
+F 2 "" H 5150 1150 50  0001 L CIN
+F 3 "https://www.mouser.com/datasheet/2/657/power-plus-dc-series-100-dc-panel-mount-1370752.pdf" H 5325 1350 50  0001 L CNN
 	1    5350 1350
 	1    0    0    -1

Commit message: Add IMU breakout board
Connections:
- wire segments 113 -> 125
Changed lines of the file:
@@
 $Descr A4 11693 8268
 encoding utf-8
-Sheet 1 2
+Sheet 1 3
 Title "Prototype E-board Schematic"
 Date ""
@@
 Connection ~ 2200 2200
 Wire Wire Line
-	3750 2650 4300 2650
-Wire Wire Line
-	3750 2750 4300 2750
+	3750 2650 4000 2650
 $Comp
 L power:GNDD #PWR020
@@
 Wire Wire Line
 	1300 2600 1450 2600
+$Sheet
+S 4300 3550 550  700
+U 5DAF980D
+F0 "SparkfunMP6050Breakout" 50
+F1 "MP6050.sch" 50
+F2 "VCC" I L 4300 3650 50
+F3 "GND" I L 4300 4150 50
+F4 "INT" I L 4300 4050 50
+F5 "SCL" I L 4300 3950 50
+F6 "SDA" I L 4300 3850 50
+F7 "VIO" I L 4300 3750 50
+$EndSheet
+$Comp
+L power:+5V #PWR?
+U 1 1 5DB03923
+P 4100 3650
+F 0 "#PWR?" H 4100 3500 50  0001 C CNN
+F 1 "+5V" H 4100 3790 50  0000 C CNN
+F 2 "" H 4100 3650 50  0001 C CNN
+F 3 "" H 4100 3650 50  0001 C CNN
+	1    4100 3650
+	1    0    0    -1
+$EndComp
+Wire Wire Line
+	4100 3650 4150 3650
+Wire Wire Line
+	4150 3650 4150 3750
+Wire Wire Line
+	4150 3750 4300 3750
+Connection ~ 4150 3650
+Wire Wire Line
+	4150 3650 4300 3650
+Wire Wire Line
+	3750 2750 3900 2750
+Wire Wire Line
+	4300 3850 4000 3850
+Wire Wire Line
+	4000 3850 4000 2650
+Connection ~ 4000 2650
+Wire Wire Line
+	4000 2650 4300 2650
+Wire Wire Line
+	3900 2750 3900 3950
+Wire Wire Line
+	3900 3950 4300 3950
+Connection ~ 3900 2750
+Wire Wire Line
+	3900 2750 4300 2750
+Wire Wire Line
+	3750 4050 4300 4050
+$Comp
+L power:GNDD #PWR?
+U 1 1 5DB1BAC9
+P 4150 4150
+F 0 "#PWR?" H 4150 3900 50  0001 C CNN
+F 1 "GNDD" H 4150 4025 50  0000 C CNN
+F 2 "" H 4150 4150 50  0001 C CNN
+F 3 "" H 4150 4150 50  0001 C CNN
+	1    4150 4150
+	1    0    0    -1
+$EndComp
+Wire Wire Line
+	4150 4150 4300 4150
 Wire Bus Line
 	5600 2400 5600 4850
