File: kicad-eboard/kicad-eboard.sch (KiCad schematic (older format))
At the start: 96 parts, among them SW1 ESTOP, SW2 REMOTE, SW3 POWER, U1 TinkerBoard, U2 WattMeter, U3 DC100D100CH, U4 Hokuyo_UST-10LX, U5 Hokuyo_UST-10LX, U6 PDQ15-Q24-S12-D, U7 PDQ30-Q24-S5-D

Commit message: Annotate, tweak positions
Parts:
- removed SW? (x4): AMT10_Encoder, symbol 2019Spacehawks:AMT10_Encoder
- added SW? (x4): AMT10_Encoder, symbol 2019Spacehawks:AMT10_Encoder
- gave numbers to parts that had none: 66

Commit message: Add test points
Parts:
- added TP1, TP2, TP3, TP4, TP5, TP6, TP7, TP8: TestPoint, symbol Connector:TestPoint
- gave numbers to parts that had none: 4
Connections:
- wire segments 263 -> 266
Changed lines of the file:
@@
 EESchema Schematic File Version 4
+LIBS:kicad-eboard-cache
 EELAYER 30 0
 EELAYER END
@@
 	1    0    0    -1
 $EndComp
-$Comp
-L power:GNDPWR #PWR014
-U 1 1 5D9E3FC6
-P 8650 1100
-F 0 "#PWR014" H 8650 900 50  0001 C CNN
-F 1 "GNDPWR" H 8654 946 50  0000 C CNN
-F 2 "" H 8650 1050 50  0001 C CNN
-F 3 "" H 8650 1050 50  0001 C CNN
-	1    8650 1100
-	1    0    0    -1
-$EndComp
 Wire Wire Line
 	9850 950  10000 950
@@
 	4800 1200 4800 1450
 Wire Wire Line
-	3200 2650 3650 2650
+	3200 2650 3350 2650
 Wire Wire Line
-	3200 2750 3650 2750
+	3200 2750 3500 2750
 NoConn ~ 3200 3200
 Wire Wire Line
@@
 Connection ~ 4300 3850
 Wire Wire Line
-	4300 3850 3700 3850
+	4300 3850 4150 3850
 Wire Wire Line
 	4300 3850 4800 3850
@@
 AR Path="/5DFA76F5/5DE14C37" Ref="SW?"  Part="1"
 AR Path="/5DFB097B/5DE14C37" Ref="SW?"  Part="1"
-AR Path="/5DE14C37" Ref="SW?"  Part="1"
-F 0 "SW?" H 6825 3125 50  0000 C CNN
+AR Path="/5DE14C37" Ref="SW7"  Part="1"
+F 0 "SW7" H 6825 3125 50  0000 C CNN
 F 1 "AMT10_Encoder" H 6500 3200 50  0000 C CNN
 F 2 "" H 6275 2810 50  0001 C CNN
@@
 AR Path="/5DFA76F5/5DE14D39" Ref="SW?"  Part="1"
 AR Path="/5DFB097B/5DE14D39" Ref="SW?"  Part="1"
-AR Path="/5DE14D39" Ref="SW?"  Part="1"
-F 0 "SW?" H 6825 3725 50  0000 C CNN
+AR Path="/5DE14D39" Ref="SW8"  Part="1"
+F 0 "SW8" H 6825 3725 50  0000 C CNN
 F 1 "AMT10_Encoder" H 6500 3800 50  0000 C CNN
 F 2 "" H 6275 3410 50  0001 C CNN
@@
 AR Path="/5DFA76F5/5DE14E3D" Ref="SW?"  Part="1"
 AR Path="/5DFB097B/5DE14E3D" Ref="SW?"  Part="1"
-AR Path="/5DE14E3D" Ref="SW?"  Part="1"
-F 0 "SW?" H 6825 4325 50  0000 C CNN
+AR Path="/5DE14E3D" Ref="SW9"  Part="1"
+F 0 "SW9" H 6825 4325 50  0000 C CNN
 F 1 "AMT10_Encoder" H 6500 4400 50  0000 C CNN
 F 2 "" H 6275 4010 50  0001 C CNN
@@
 AR Path="/5DFA76F5/5DE14F47" Ref="SW?"  Part="1"
 AR Path="/5DFB097B/5DE14F47" Ref="SW?"  Part="1"
-AR Path="/5DE14F47" Ref="SW?"  Part="1"
-F 0 "SW?" H 6825 4925 50  0000 C CNN
+AR Path="/5DE14F47" Ref="SW10"  Part="1"
+F 0 "SW10" H 6825 4925 50  0000 C CNN
 F 1 "AMT10_Encoder" H 6500 5000 50  0000 C CNN
 F 2 "" H 6275 4610 50  0001 C CNN
@@
 	-1   0    0    -1
 $EndComp
+$Comp
+L Connector:TestPoint TP4
+U 1 1 5DC9EF3C
+P 7550 700
+F 0 "TP4" H 7608 818 50  0000 L CNN
+F 1 "TestPoint" H 7608 727 50  0000 L CNN
+F 2 "" H 7750 700 50  0001 C CNN
+F 3 "~" H 7750 700 50  0001 C CNN
+	1    7550 700
+	1    0    0    -1
+$EndComp
+$Comp
+L power:GNDPWR #PWR014
+U 1 1 5DCA0FF7
+P 7550 700
+F 0 "#PWR014" H 7550 500 50  0001 C CNN
+F 1 "GNDPWR" H 7554 546 50  0000 C CNN
+F 2 "" H 7550 650 50  0001 C CNN
+F 3 "" H 7550 650 50  0001 C CNN
+	1    7550 700
+	1    0    0    -1
+$EndComp
+$Comp
+L power:+BATT #PWR065
+U 1 1 5DCA1541
+P 7550 1100
+F 0 "#PWR065" H 7550 950 50  0001 C CNN
+F 1 "+BATT" H 7565 1273 50  0000 C CNN
+F 2 "" H 7550 1100 50  0001 C CNN
+F 3 "" H 7550 1100 50  0001 C CNN
+	1    7550 1100
+	1    0    0    -1
+$EndComp
+$Comp
+L power:+12V #PWR066
+U 1 1 5DCA1D04
+P 7550 1500
+F 0 "#PWR066" H 7550 1350 50  0001 C CNN
+F 1 "+12V" H 7550 1640 50  0000 C CNN
+F 2 "" H 7550 1500 50  0001 C CNN
+F 3 "" H 7550 1500 50  0001 C CNN
+	1    7550 1500
+	1    0    0    -1
+$EndComp
+$Comp
+L power:+5V #PWR067
+U 1 1 5DCA200F
+P 8000 650
+F 0 "#PWR067" H 8000 500 50  0001 C CNN
+F 1 "+5V" H 8000 790 50  0000 C CNN
+F 2 "" H 8000 650 50  0001 C CNN
+F 3 "" H 8000 650 50  0001 C CNN
+	1    8000 650
+	1    0    0    -1
+$EndComp
+$Comp
+L power:+3.3V #PWR068
+U 1 1 5DCA23FA
+P 8000 1100
+F 0 "#PWR068" H 8000 950 50  0001 C CNN
+F 1 "+3.3V" H 8000 1240 50  0000 C CNN
+F 2 "" H 8000 1100 50  0001 C CNN
+F 3 "" H 8000 1100 50  0001 C CNN
+	1    8000 1100
+	1    0    0    -1
+$EndComp
+$Comp
+L power:GNDPWR #PWR069
+U 1 1 5DCBA260
+P 8650 1100
+F 0 "#PWR069" H 8650 900 50  0001 C CNN
+F 1 "GNDPWR" H 8654 946 50  0000 C CNN
+F 2 "" H 8650 1050 50  0001 C CNN
+F 3 "" H 8650 1050 50  0001 C CNN
+	1    8650 1100
+	1    0    0    -1
+$EndComp
+$Comp
+L Connector:TestPoint TP7
+U 1 1 5DCBC539
+P 8000 650
+F 0 "TP7" H 7942 676 50  0000 R CNN
+F 1 "TestPoint" H 7942 767 50  0000 R CNN
+F 2 "" H 8200 650 50  0001 C CNN
+F 3 "~" H 8200 650 50  0001 C CNN
+	1    8000 650
+	-1   0    0    1
+$EndComp
+$Comp
+L Connector:TestPoint TP8
+U 1 1 5DCBC74F
+P 8000 1100
+F 0 "TP8" H 7942 1126 50  0000 R CNN
+F 1 "TestPoint" H 7942 1217 50  0000 R CNN
+F 2 "" H 8200 1100 50  0001 C CNN
+F 3 "~" H 8200 1100 50  0001 C CNN
+	1    8000 1100
+	-1   0    0    1
+$EndComp
+$Comp
+L Connector:TestPoint TP6
+U 1 1 5DCBC301
+P 7550 1500
+F 0 "TP6" H 7492 1526 50  0000 R CNN
+F 1 "TestPoint" H 7492 1617 50  0000 R CNN
+F 2 "" H 7750 1500 50  0001 C CNN
+F 3 "~" H 7750 1500 50  0001 C CNN
+	1    7550 1500
+	-1   0    0    1
+$EndComp
+$Comp
+L Connector:TestPoint TP5
+U 1 1 5DCA1990
+P 7550 1100
+F 0 "TP5" H 7492 1126 50  0000 R CNN
+F 1 "TestPoint" H 7492 1217 50  0000 R CNN
+F 2 "" H 7750 1100 50  0001 C CNN
+F 3 "~" H 7750 1100 50  0001 C CNN
+	1    7550 1100
+	-1   0    0    1
+$EndComp
+$Comp
+L Connector:TestPoint TP3
+U 1 1 5DD30A1C
+P 4150 3850
+F 0 "TP3" H 4092 3876 50  0000 R CNN
+F 1 "TestPoint" H 4092 3967 50  0000 R CNN
+F 2 "" H 4350 3850 50  0001 C CNN
+F 3 "~" H 4350 3850 50  0001 C CNN
+	1    4150 3850
+	1    0    0    -1
+$EndComp
+Connection ~ 4150 3850
+Wire Wire Line
+	4150 3850 3700 3850
+$Comp
+L Connector:TestPoint TP1
+U 1 1 5DD312C3
+P 3350 2650
+F 0 "TP1" H 3292 2676 50  0000 R CNN
+F 1 "TestPoint" H 3292 2767 50  0000 R CNN
+F 2 "" H 3550 2650 50  0001 C CNN
+F 3 "~" H 3550 2650 50  0001 C CNN
+	1    3350 2650
+	1    0    0    -1
+$EndComp
+Connection ~ 3350 2650
+Wire Wire Line
+	3350 2650 3650 2650
+$Comp
+L Connector:TestPoint TP2
+U 1 1 5DD318AA
+P 3500 2750
+F 0 "TP2" H 3442 2776 50  0000 R CNN
+F 1 "TestPoint" H 3442 2867 50  0000 R CNN
+F 2 "" H 3700 2750 50  0001 C CNN
+F 3 "~" H 3700 2750 50  0001 C CNN
+	1    3500 2750
+	1    0    0    -1
+$EndComp
+Connection ~ 3500 2750
+Wire Wire Line
+	3500 2750 3650 2750
 $EndSCHEMATC

Commit message: Use 91k resistors instead of two 47k to fit parts on hand
Parts:
- removed R33, R34, R35, R36, R37, R38, R39, R40, R41, R42, R43, R44, R45, R46, R47: 47K, symbol Device:R
- R18, R19, R20, R21, R22, R23, R24, R25, R26, R27, R28, R29, R30, R31, R32: value 47K -> 91K

Commit message: Add some footprints
Parts:
- BT1, BT2: value Battery -> #Battery
- C1, C5, C6, C7, C8: footprint (none) -> Capacitor_THT:CP_Radial_D5.0mm_P2.50mm
- C10, C2, C9: footprint (none) -> Capacitor_SMD:C_0805_2012Metric_Pad1.15x1.40mm_HandSolder
- CB1: value MRCB_187080F-03-1 -> #MRCB_187080F-03-1
- L1, L2: footprint (none) -> Inductor_SMD:L_1206_3216Metric
- M1, M2, M3, M4: value Motor_DC -> #Motor_DC
- M5: value Digger_Motor -> #Digger_Motor
- M6, M7, M8, M9: value Lin_Actuator -> #Lin_Actuator
- MES1: value Voltmeter_DC -> #Voltmeter_DC
- R10, R11, R12, R13, R14, R15, R16, R17, R18, R19, R20, R21, R22, R23, R24, R25, R26, R27, R28, R29, R3, R30, R31, R32, R4, R5, R6, R7, R8, R9: footprint (none) -> Resistor_SMD:R_0603_1608Metric_Pad1.05x0.95mm_HandSolder
- RV1, RV2: footprint (none) -> Potentiometer_THT:Potentiometer_Piher_PT-10-V05_Vertical
- RV3: footprint (none) -> Connector_JST:JST_XH_B2B-XH-AM_1x02_P2.50mm_Vertical
- RV4, RV5, RV6, SW4, SW5: footprint (none) -> Connector_JST:JST_XH_B3B-XH-A_1x03_P2.50mm_Vertical
- SW1: value ESTOP -> #ESTOP
- SW10, SW6, SW7, SW8, SW9: footprint (none) -> Connector_JST:JST_XH_B5B-XH-A_1x05_P2.50mm_Vertical
- SW2: value REMOTE -> #REMOTE
- SW3: value POWER -> #POWER
- TP1, TP2, TP3, TP4, TP5, TP6, TP7, TP8: footprint (none) -> TestPoint:TestPoint_Bridge_Pitch2.54mm_Drill1.0mm
- U1: footprint (none) -> Connector_IDC:IDC-Header_2x20_P2.54mm_Vertical
- U10, U11, U12, U13, U4, U5, U8: footprint (none) -> Connector_JST:JST_XH_B2B-XH-A_1x02_P2.50mm_Vertical
- U2: value WattMeter -> #WattMeter
- U3: value DC100D100CH -> #DC100D100CH

Commit message: Add footprints for DC-DC converters
Parts:
- C1, C7, C8: footprint Capacitor_THT:CP_Radial_D5.0mm_P2.50mm -> Capacitor_SMD:C_0603_1608Metric_Pad1.05x0.95mm_HandSolder
- U6, U7: footprint (none) -> 2019Spacehawks:PDQXX-D_DC-DC_converter
Changed lines of the file:
@@
 F 0 "U6" H 10650 1450 50  0000 C CNN
 F 1 "PDQ15-Q24-S12-D" H 10400 1350 50  0000 C CNN
-F 2 "" H 10350 900 50  0001 C CNN
+F 2 "2019Spacehawks:PDQXX-D_DC-DC_converter" H 10350 900 50  0001 C CNN
 F 3 "https://www.cui.com/product/resource/pdq15-d.pdf" H 10450 1000 50  0001 C CNN
 F 4 "12V" H 10600 1250 50  0000 C CNN "Vout"
@@
 F 0 "U7" H 10650 2450 50  0000 C CNN
 F 1 "PDQ30-Q24-S5-D" H 10400 2350 50  0000 C CNN
-F 2 "" H 10350 1900 50  0001 C CNN
+F 2 "2019Spacehawks:PDQXX-D_DC-DC_converter" H 10350 1900 50  0001 C CNN
 F 3 "https://www.cui.com/product/resource/pdq30-d.pdf" H 10450 2000 50  0001 C CNN
 F 4 "5V" H 10600 2250 50  0000 C CNN "Vout"
@@
 F 0 "C7" H 9425 1050 50  0000 L CNN
 F 1 "1u" H 9425 850 50  0000 L CNN
-F 2 "Capacitor_THT:CP_Radial_D5.0mm_P2.50mm" H 9438 800 50  0001 C CNN
+F 2 "Capacitor_SMD:C_0603_1608Metric_Pad1.05x0.95mm_HandSolder" H 9438 800 50  0001 C CNN
 F 3 "~" H 9400 950 50  0001 C CNN
 	1    9400 950
@@
 F 0 "C8" H 9425 2050 50  0000 L CNN
 F 1 "1u" H 9425 1850 50  0000 L CNN
-F 2 "Capacitor_THT:CP_Radial_D5.0mm_P2.50mm" H 9438 1800 50  0001 C CNN
+F 2 "Capacitor_SMD:C_0603_1608Metric_Pad1.05x0.95mm_HandSolder" H 9438 1800 50  0001 C CNN
 F 3 "~" H 9400 1950 50  0001 C CNN
 	1    9400 1950
@@
 F 0 "C1" H 625 2850 50  0000 L CNN
 F 1 "1u" H 625 2650 50  0000 L CNN
-F 2 "Capacitor_THT:CP_Radial_D5.0mm_P2.50mm" H 638 2600 50  0001 C CNN
+F 2 "Capacitor_SMD:C_0603_1608Metric_Pad1.05x0.95mm_HandSolder" H 638 2600 50  0001 C CNN
 F 3 "~" H 600 2750 50  0001 C CNN
 	1    600  2750

Commit message: Add more test points, battary->PCB connector
Parts:
- added J1: Conn_01x02, Connector_JST:JST_XH_B2B-XH-A_1x02_P2.50mm_Vertical, symbol Connector_Generic:Conn_01x02
- added TP10, TP9: TestPoint, TestPoint:TestPoint_Bridge_Pitch2.54mm_Drill1.0mm, symbol Connector:TestPoint
Connections:
- wire segments 266 -> 268
Other:
- note added: "Ports & Test Points"
- note added: "Power (off PCB)"
- moved on the sheet: BT1, BT2, CB1, SW1, U2, U3

Commit message: Move #s to actually work
Parts:
- removed BT1, BT2: #Battery, symbol Device:Battery
- removed CB1: #MRCB_187080F-03-1, symbol Device:CircuitBreaker_1P
- removed M1, M2, M3, M4: #Motor_DC, symbol Motor:Motor_DC
- removed M5: #Digger_Motor, symbol Motor:Motor_DC
- removed M6, M7, M8, M9: #Lin_Actuator, symbol Motor:Motor_DC
- removed MES1: #Voltmeter_DC, symbol Device:Voltmeter_DC
- removed SW1: #ESTOP, symbol Switch:SW_SPST
- removed SW2: #REMOTE, symbol 2019Spacehawks:Wireless_Relay
- removed SW3: #POWER, symbol 2019Spacehawks:SW_SPST_LED
- removed U2: #WattMeter, symbol 2019Spacehawks:WattMeter
- removed U3: #DC100D100CH, symbol Relay_SolidState:34.81-8240
Connections:
- net labels added: #DC100D100CH, #POWER, #REMOTE, #Voltmeter_DC, Battery, Digger_Motor, ESTOP, Lin_Actuator, MRCB_187080F-03-1, Motor_DC, WattMeter
Changed lines of the file:
@@
 $EndDescr
 $Comp
-L Device:Battery BT1
+L Device:Battery #BT1
 U 1 1 5D911E0B
 P 600 1150
-F 0 "BT1" H 708 1196 50  0000 L CNN
-F 1 "#Battery" H 708 1105 50  0000 L CNN
+F 0 "#BT1" H 708 1196 50  0000 L CNN
+F 1 "Battery" H 708 1105 50  0000 L CNN
 F 2 "" V 600 1210 50  0001 C CNN
 F 3 "~" V 600 1210 50  0001 C CNN
@@
 $EndComp
 $Comp
-L Device:CircuitBreaker_1P CB1
+L Device:CircuitBreaker_1P #CB1
 U 1 1 5D911FF4
 P 1500 950
-F 0 "CB1" V 1235 950 50  0000 C CNN
-F 1 "#MRCB_187080F-03-1" V 1326 950 50  0000 C CNN
+F 0 "#CB1" V 1235 950 50  0000 C CNN
+F 1 "MRCB_187080F-03-1" V 1326 950 50  0000 C CNN
 F 2 "" H 1500 950 50  0001 C CNN
 F 3 "https://www.solar-electric.com/lib/wind-sun/Bussmann-MRCB.pdf" H 1500 950 50  0001 C CNN
@@
 $EndComp
 $Comp
-L 2019Spacehawks:WattMeter U2
+L 2019Spacehawks:WattMeter #U2
 U 1 1 5D9123C3
 P 2450 1100
-F 0 "U2" H 2450 1425 50  0000 C CNN
-F 1 "#WattMeter" H 2450 1334 50  0000 C CNN
+F 0 "#U2" H 2450 1425 50  0000 C CNN
+F 1 "WattMeter" H 2450 1334 50  0000 C CNN
 F 2 "" H 2450 1100 50  0001 C CNN
 F 3 "" H 2450 1100 50  0001 C CNN
@@
 	2050 1350 1100 1350
 $Comp
-L Relay_SolidState:34.81-8240 U3
+L Relay_SolidState:34.81-8240 #U3
 U 1 1 5D913EE3
 P 5000 1100
-F 0 "U3" H 5000 1425 50  0000 C CNN
+F 0 "#U3" H 5000 1425 50  0000 C CNN
 F 1 "#DC100D100CH" H 5000 1334 50  0000 C CNN
 F 2 "" H 4800 900 50  0001 L CIN
@@
 $EndComp
 $Comp
-L Switch:SW_SPST SW1
+L Switch:SW_SPST #SW1
 U 1 1 5D914CA6
 P 3200 900
-F 0 "SW1" H 3200 1135 50  0000 C CNN
-F 1 "#ESTOP" H 3200 1044 50  0000 C CNN
+F 0 "#SW1" H 3200 1135 50  0000 C CNN
+F 1 "ESTOP" H 3200 1044 50  0000 C CNN
 F 2 "" H 3200 900 50  0001 C CNN
 F 3 "" H 3200 900 50  0001 C CNN
@@
 	5300 600  5300 1000
 $Comp
-L Device:Battery BT2
+L Device:Battery #BT2
 U 1 1 5D9D77E5
 P 1100 1150
-F 0 "BT2" H 1208 1196 50  0000 L CNN
-F 1 "#Battery" H 1208 1105 50  0000 L CNN
+F 0 "#BT2" H 1208 1196 50  0000 L CNN
+F 1 "Battery" H 1208 1105 50  0000 L CNN
 F 2 "" V 1100 1210 50  0001 C CNN
 F 3 "~" V 1100 1210 50  0001 C CNN
@@
 	700  1350 600  1350
 $Comp
-L Device:Voltmeter_DC MES1
+L Device:Voltmeter_DC #MES1
 U 1 1 5DA52428
 P 6600 1050
-F 0 "MES1" H 6470 1090 50  0000 R CNN
+F 0 "#MES1" H 6470 1090 50  0000 R CNN
 F 1 "#Voltmeter_DC" H 6470 1020 50  0000 R CNN
 F 2 "" V 6600 1150 50  0001 C CNN
@@
 	3200 2500 3300 2500
 $Comp
-L 2019Spacehawks:Wireless_Relay SW2
+L 2019Spacehawks:Wireless_Relay #SW2
 U 1 1 5DB15C61
 P 3700 900
-F 0 "SW2" H 3800 1100 50  0000 C CNN
+F 0 "#SW2" H 3800 1100 50  0000 C CNN
 F 1 "#REMOTE" H 3700 700 50  0000 C CNN
 F 2 "" H 3700 900 50  0001 C CNN
@@
 	4650 1200 4450 1200
 $Comp
-L 2019Spacehawks:SW_SPST_LED SW3
+L 2019Spacehawks:SW_SPST_LED #SW3
 U 1 1 5DBF72D0
 P 4250 900
-F 0 "SW3" H 4275 1125 50  0000 L CNN
+F 0 "#SW3" H 4275 1125 50  0000 L CNN
 F 1 "#POWER" H 4250 725 50  0000 C CNN
 F 2 "" H 4250 1200 50  0001 C CNN
@@
 Wire Wire Line
 	5750 3150 5950 3150
-$Comp
-L 2019Spacehawks:Sabertooth2x60 U?
-U 1 1 5DDDCDE4
-P 5300 2500
-AR Path="/5D9AC27F/5DDDCDE4" Ref="U?"  Part="1"
-AR Path="/5D9BDACA/5DDDCDE4" Ref="U?"  Part="1"
-AR Path="/5D981157/5DDDCDE4" Ref="U?"  Part="1"
-AR Path="/5D9ACC15/5DDDCDE4" Ref="U?"  Part="1"
-AR Path="/5D9ACC1B/5DDDCDE4" Ref="U?"  Part="1"
-AR Path="/5D9B81A1/5DDDCDE4" Ref="U?"  Part="1"
-AR Path="/5D9B81A7/5DDDCDE4" Ref="U?"  Part="1"
-AR Path="/5DFA76F5/5DDDCDE4" Ref="U?"  Part="1"
-AR Path="/5DFB097B/5DDDCDE4" Ref="U?"  Part="1"
-AR Path="/5DDDCDE4" Ref="U8"  Part="1"
-F 0 "U8" H 5500 2800 50  0000 C CNN
-F 1 "Sabertooth2x60" H 5250 2700 50  0000 C CNN
-F 2 "Connector_JST:JST_XH_B2B-XH-A_1x02_P2.50mm_Vertical" H 5300 2500 50  0001 C CNN
-F 3 "" H 5300 2500 50  0001 C CNN
-	1    5300 2500
-	1    0    0    -1
-$EndComp
 NoConn ~ 4800 2750
 $Comp
@@
 	5750 5150 5950 5150
 $Comp
-L Motor:Motor_DC M6
+L Motor:Motor_DC #M6
 U 1 1 5E53431B
 P 5950 5350
-F 0 "M6" H 6050 5100 50  0000 L CNN
-F 1 "#Lin_Actuator" H 5700 5050 50  0000 L TNN
+F 0 "#M6" H 6050 5100 50  0000 L CNN
+F 1 "Lin_Actuator" H 5700 5050 50  0000 L TNN
 F 2 "" H 5950 5260 50  0001 C CNN
 F 3 "https://cdn.shopify.com/s/files/1/0615/2193/files/firgelli-feedback-rod-linear-actuator-spec-sheet.pdf?88045" H 5950 5260 50  0001 C CNN
@@
 	3600 5200 3200 5200
 $Comp
-L Motor:Motor_DC M7
+L Motor:Motor_DC #M7
 U 1 1 5EA9C69C
 P 5950 5950
-F 0 "M7" H 6050 5700 50  0000 L CNN
-F 1 "#Lin_Actuator" H 5700 5650 50  0000 L TNN
+F 0 "#M7" H 6050 5700 50  0000 L CNN
+F 1 "Lin_Actuator" H 5700 5650 50  0000 L TNN
 F 2 "" H 5950 5860 50  0001 C CNN
 F 3 "https://cdn.shopify.com/s/files/1/0615/2193/files/firgelli-feedback-rod-linear-actuator-spec-sheet.pdf?88045" H 5950 5860 50  0001 C CNN
@@
 $EndComp
 $Comp
-L Motor:Motor_DC M8
+L Motor:Motor_DC #M8
 U 1 1 5EA9CC29
 P 5950 6600
-F 0 "M8" H 6050 6350 50  0000 L CNN
-F 1 "#Lin_Actuator" H 5700 6300 50  0000 L TNN
+F 0 "#M8" H 6050 6350 50  0000 L CNN
+F 1 "Lin_Actuator" H 5700 6300 50  0000 L TNN
 F 2 "" H 5950 6510 50  0001 C CNN
 F 3 "https://cdn.shopify.com/s/files/1/0615/2193/files/firgelli-feedback-rod-linear-actuator-spec-sheet.pdf?88045" H 5950 6510 50  0001 C CNN
@@
 $EndComp
 $Comp
-L Motor:Motor_DC M9
+L Motor:Motor_DC #M9
 U 1 1 5EA9CD19
 P 5950 7200
-F 0 "M9" H 6050 6950 50  0000 L CNN
-F 1 "#Lin_Actuator" H 5700 6900 50  0000 L TNN
+F 0 "#M9" H 6050 6950 50  0000 L CNN
+F 1 "Lin_Actuator" H 5700 6900 50  0000 L TNN
 F 2 "" H 5950 7110 50  0001 C CNN
 F 3 "https://cdn.shopify.com/s/files/1/0615/2193/files/firgelli-feedback-rod-linear-actuator-spec-sheet.pdf?88045" H 5950 7110 50  0001 C CNN
@@
 AR Path="/5DFA76F5/5EB6AEB7" Ref="M?"  Part="1"
 AR Path="/5DFB097B/5EB6AEB7" Ref="M?"  Part="1"
-AR Path="/5EB6AEB7" Ref="M5"  Part="1"
-F 0 "M5" H 6000 4750 50  0000 L CNN
-F 1 "#Digger_Motor" H 5700 4350 50  0000 L TNN
+AR Path="/5EB6AEB7" Ref="#M5"  Part="1"
+F 0 "#M5" H 6000 4750 50  0000 L CNN
+F 1 "Digger_Motor" H 5700 4350 50  0000 L TNN
 F 2 "" H 5950 4560 50  0001 C CNN
 F 3 "~" H 5950 4560 50  0001 C CNN
@@
 AR Path="/5DFA76F5/5EB988EA" Ref="M?"  Part="1"
 AR Path="/5DFB097B/5EB988EA" Ref="M?"  Part="1"
-AR Path="/5EB988EA" Ref="M1"  Part="1"
-F 0 "M1" H 6000 2350 50  0000 L CNN
-F 1 "#Motor_DC" H 5700 1950 50  0000 L TNN
+AR Path="/5EB988EA" Ref="#M1"  Part="1"
+F 0 "#M1" H 6000 2350 50  0000 L CNN
+F 1 "Motor_DC" H 5700 1950 50  0000 L TNN
 F 2 "" H 5950 2160 50  0001 C CNN
 F 3 "~" H 5950 2160 50  0001 C CNN
@@
 AR Path="/5DFA76F5/5EB98646" Ref="M?"  Part="1"
 AR Path="/5DFB097B/5EB98646" Ref="M?"  Part="1"
-AR Path="/5EB98646" Ref="M4"  Part="1"
-F 0 "M4" H 6000 4150 50  0000 L CNN
-F 1 "#Motor_DC" H 5700 3750 50  0000 L TNN
+AR Path="/5EB98646" Ref="#M4"  Part="1"
+F 0 "#M4" H 6000 4150 50  0000 L CNN
+F 1 "Motor_DC" H 5700 3750 50  0000 L TNN
 F 2 "" H 5950 3960 50  0001 C CNN
 F 3 "~" H 5950 3960 50  0001 C CNN
@@
 AR Path="/5DFA76F5/5EB98726" Ref="M?"  Part="1"
 AR Path="/5DFB097B/5EB98726" Ref="M?"  Part="1"
-AR Path="/5EB98726" Ref="M3"  Part="1"
-F 0 "M3" H 6000 3550 50  0000 L CNN
-F 1 "#Motor_DC" H 5700 3150 50  0000 L TNN
+AR Path="/5EB98726" Ref="#M3"  Part="1"
+F 0 "#M3" H 6000 3550 50  0000 L CNN
+F 1 "Motor_DC" H 5700 3150 50  0000 L TNN
 F 2 "" H 5950 3360 50  0001 C CNN
 F 3 "~" H 5950 3360 50  0001 C CNN
@@
 AR Path="/5DFA76F5/5EB98806" Ref="M?"  Part="1"
 AR Path="/5DFB097B/5EB98806" Ref="M?"  Part="1"
-AR Path="/5EB98806" Ref="M2"  Part="1"
-F 0 "M2" H 6000 2950 50  0000 L CNN
-F 1 "#Motor_DC" H 5700 2550 50  0000 L TNN
+AR Path="/5EB98806" Ref="#M2"  Part="1"
+F 0 "#M2" H 6000 2950 50  0000 L CNN
+F 1 "Motor_DC" H 5700 2550 50  0000 L TNN
 F 2 "" H 5950 2760 50  0001 C CNN
 F 3 "~" H 5950 2760 50  0001 C CNN
@@
 Wire Notes Line
 	8900 5350 11200 5350
+$Comp
+L 2019Spacehawks:Sabertooth2x60 U?
+U 1 1 5DDDCDE4
+P 5300 2500
+AR Path="/5D9AC27F/5DDDCDE4" Ref="U?"  Part="1"
+AR Path="/5D9BDACA/5DDDCDE4" Ref="U?"  Part="1"
+AR Path="/5D981157/5DDDCDE4" Ref="U?"  Part="1"
+AR Path="/5D9ACC15/5DDDCDE4" Ref="U?"  Part="1"
+AR Path="/5D9ACC1B/5DDDCDE4" Ref="U?"  Part="1"
+AR Path="/5D9B81A1/5DDDCDE4" Ref="U?"  Part="1"
+AR Path="/5D9B81A7/5DDDCDE4" Ref="U?"  Part="1"
+AR Path="/5DFA76F5/5DDDCDE4" Ref="U?"  Part="1"
+AR Path="/5DFB097B/5DDDCDE4" Ref="U?"  Part="1"
+AR Path="/5DDDCDE4" Ref="U8"  Part="1"
+F 0 "U8" H 5500 2800 50  0000 C CNN
+F 1 "Sabertooth2x60" H 5250 2700 50  0000 C CNN
+F 2 "Connector_JST:JST_XH_B2B-XH-A_1x02_P2.50mm_Vertical" H 5300 2500 50  0001 C CNN
+F 3 "" H 5300 2500 50  0001 C CNN
+	1    5300 2500
+	1    0    0    -1
+$EndComp
 $EndSCHEMATC
