File: kicad-eboard/kicad-eboard.sch (KiCad schematic (older format))
At the start: 79 parts, among them J1 Conn_01x02, J2 Conn_02x03, M1 Hopper_Servo, SW1 SRX_Encoder, SW4 LIMIT_1, SW5 LIMIT_2, U1 TinkerBoard, U10 Sabertooth2x60, U11 Sabertooth2x60, U12 Sabertooth2x60, U13 INA4181, U14 MCP3008, U15 REF2033, U2 ADS1015IDGS, U3 INA4181, U4 Hokuyo_UST-10LX, U5 Hokuyo_UST-10LX, U6 PDQ15-Q24-S12-D, U7 PDQ30-Q24-S5-D, U8 Sabertooth2x60

Commit message: Add 1.65 TP
Parts:
- added TP?: TestPoint, TestPoint:TestPoint_Bridge_Pitch2.54mm_Drill1.0mm, symbol Connector:TestPoint
Changed lines of the file:
@@
 	1    0    0    -1
 $EndComp
+$Comp
+L 2019Spacehawks:+1.65V #PWR?
+U 1 1 5EA3169F
+P 9650 5150
+F 0 "#PWR?" H 9650 5000 50  0001 C CNN
+F 1 "+1.65V" H 9650 5290 50  0000 C CNN
+F 2 "" H 9650 5150 50  0001 C CNN
+F 3 "" H 9650 5150 50  0001 C CNN
+	1    9650 5150
+	1    0    0    -1
+$EndComp
+$Comp
+L Connector:TestPoint TP?
+U 1 1 5EA31926
+P 9650 5150
+F 0 "TP?" H 9592 5176 50  0000 R CNN
+F 1 "TestPoint" H 9592 5267 50  0000 R CNN
+F 2 "TestPoint:TestPoint_Bridge_Pitch2.54mm_Drill1.0mm" H 9850 5150 50  0001 C CNN
+F 3 "~" H 9850 5150 50  0001 C CNN
+	1    9650 5150
+	-1   0    0    1
+$EndComp
 $EndSCHEMATC

Commit message: Add 1.65 TP
Parts:
- gave numbers to parts that had none: 1
Changed lines of the file:
@@
 $EndComp
 $Comp
-L 2019Spacehawks:+1.65V #PWR?
+L 2019Spacehawks:+1.65V #PWR0100
 U 1 1 5EA3169F
 P 9650 5150
-F 0 "#PWR?" H 9650 5000 50  0001 C CNN
+F 0 "#PWR0100" H 9650 5000 50  0001 C CNN
 F 1 "+1.65V" H 9650 5290 50  0000 C CNN
 F 2 "" H 9650 5150 50  0001 C CNN
@@
 $EndComp
 $Comp
-L Connector:TestPoint TP?
+L Connector:TestPoint TP15
 U 1 1 5EA31926
 P 9650 5150
-F 0 "TP?" H 9592 5176 50  0000 R CNN
+F 0 "TP15" H 9592 5176 50  0000 R CNN
 F 1 "TestPoint" H 9592 5267 50  0000 R CNN
 F 2 "TestPoint:TestPoint_Bridge_Pitch2.54mm_Drill1.0mm" H 9850 5150 50  0001 C CNN

Commit message: Separate analog/digital ground, Vref
Parts:
- added NT?: Net-Tie_2, symbol Device:Net-Tie_2
Connections:
- net labels added: +3.3VADC, GNDREF
- wire segments 318 -> 324
- no-connect marks 28 -> 27
Changed lines of the file:
@@
 	8700 2700 8750 2700
-$Comp
-L power:GNDD #PWR081
-U 1 1 5FAF482E
-P 9050 3000
-F 0 "#PWR081" H 9050 2750 50  0001 C CNN
-F 1 "GNDD" H 9050 2875 50  0000 C CNN
-F 2 "" H 9050 3000 50  0001 C CNN
-F 3 "" H 9050 3000 50  0001 C CNN
-	1    9050 3000
-	1    0    0    -1
-$EndComp
 $Comp
 L 2019Spacehawks:+1.65V #PWR082
@@
 Wire Wire Line
 	9500 2650 9450 2650
-NoConn ~ 9450 2800
 Text Label 5800 2200 0    50   ~ 0
 M1+
@@
 M5+
 $Comp
-L power:GNDD #PWR044
-U 1 1 5E6344DE
-P 6300 3050
-F 0 "#PWR044" H 6300 2800 50  0001 C CNN
-F 1 "GNDD" H 6300 2925 50  0000 C CNN
-F 2 "" H 6300 3050 50  0001 C CNN
-F 3 "" H 6300 3050 50  0001 C CNN
-	1    6300 3050
-	1    0    0    -1
-$EndComp
-$Comp
 L 2019Spacehawks:+1.65V #PWR055
 U 1 1 5E634864
@@
 Wire Wire Line
 	6750 2200 6750 2300
-$Comp
-L power:+3.3V #PWR043
-U 1 1 5E6A9309
-P 6300 2050
-F 0 "#PWR043" H 6300 1900 50  0001 C CNN
-F 1 "+3.3V" H 6300 2190 50  0000 C CNN
-F 2 "" H 6300 2050 50  0001 C CNN
-F 3 "" H 6300 2050 50  0001 C CNN
-	1    6300 2050
-	1    0    0    -1
-$EndComp
 $Comp
 L Device:R R8
@@
 $EndComp
 $Comp
-L power:+3.3V #PWR045
-U 1 1 5E77AB71
-P 6300 3400
-F 0 "#PWR045" H 6300 3250 50  0001 C CNN
-F 1 "+3.3V" H 6300 3540 50  0000 C CNN
-F 2 "" H 6300 3400 50  0001 C CNN
-F 3 "" H 6300 3400 50  0001 C CNN
-	1    6300 3400
-	1    0    0    -1
-$EndComp
-$Comp
-L power:GNDD #PWR046
-U 1 1 5E79847B
-P 6300 4400
-F 0 "#PWR046" H 6300 4150 50  0001 C CNN
-F 1 "GNDD" H 6300 4275 50  0000 C CNN
-F 2 "" H 6300 4400 50  0001 C CNN
-F 3 "" H 6300 4400 50  0001 C CNN
-	1    6300 4400
-	1    0    0    -1
-$EndComp
-$Comp
 L 2019Spacehawks:+1.65V #PWR054
 U 1 1 5E798796
@@
 	1    0    0    -1
 $EndComp
-$Comp
-L power:GNDD #PWR061
-U 1 1 5E83A7A3
-P 8600 4450
-F 0 "#PWR061" H 8600 4200 50  0001 C CNN
-F 1 "GNDD" H 8600 4325 50  0000 C CNN
-F 2 "" H 8600 4450 50  0001 C CNN
-F 3 "" H 8600 4450 50  0001 C CNN
-	1    8600 4450
-	1    0    0    -1
-$EndComp
-$Comp
-L power:GNDD #PWR063
-U 1 1 5E83ABC2
-P 8900 4450
-F 0 "#PWR063" H 8900 4200 50  0001 C CNN
-F 1 "GNDD" H 8900 4325 50  0000 C CNN
-F 2 "" H 8900 4450 50  0001 C CNN
-F 3 "" H 8900 4450 50  0001 C CNN
-	1    8900 4450
-	1    0    0    -1
-$EndComp
 Wire Wire Line
 	8100 4150 7450 4150
@@
 Wire Wire Line
 	7750 2900 7750 3850
-$Comp
-L power:+3.3V #PWR060
-U 1 1 5EA8797E
-P 8600 3350
-F 0 "#PWR060" H 8600 3200 50  0001 C CNN
-F 1 "+3.3V" H 8600 3490 50  0000 C CNN
-F 2 "" H 8600 3350 50  0001 C CNN
-F 3 "" H 8600 3350 50  0001 C CNN
-	1    8600 3350
-	1    0    0    -1
-$EndComp
 $Comp
 L power:+3.3V #PWR062
@@
 Wire Wire Line
 	7600 4250 8100 4250
-$Comp
-L power:GNDD #PWR059
-U 1 1 605C7D19
-P 7150 4550
-F 0 "#PWR059" H 7150 4300 50  0001 C CNN
-F 1 "GNDD" H 7150 4425 50  0000 C CNN
-F 2 "" H 7150 4550 50  0001 C CNN
-F 3 "" H 7150 4550 50  0001 C CNN
-	1    7150 4550
-	1    0    0    -1
-$EndComp
 Wire Wire Line
 	7150 4550 7150 4500
@@
 Wire Wire Line
 	7600 4550 7600 4500
-Connection ~ 7150 4550
 Wire Wire Line
 	7450 4500 7450 4550
@@
 Wire Wire Line
 	7600 2950 7600 2900
-$Comp
-L power:GNDD #PWR058
-U 1 1 60653C8F
-P 7150 3200
-F 0 "#PWR058" H 7150 2950 50  0001 C CNN
-F 1 "GNDD" H 7150 3075 50  0000 C CNN
-F 2 "" H 7150 3200 50  0001 C CNN
-F 3 "" H 7150 3200 50  0001 C CNN
-	1    7150 3200
-	1    0    0    -1
-$EndComp
 Wire Wire Line
 	7150 3200 7150 3150
@@
 Wire Wire Line
 	7600 3200 7600 3150
-Connection ~ 7150 3200
 Wire Wire Line
 	7450 3150 7450 3200
@@
 $EndComp
 $Comp
-L power:GNDD #PWR095
-U 1 1 5E769D66
-P 9350 4450
-F 0 "#PWR095" H 9350 4200 50  0001 C CNN
-F 1 "GNDD" H 9350 4325 50  0000 C CNN
-F 2 "" H 9350 4450 50  0001 C CNN
-F 3 "" H 9350 4450 50  0001 C CNN
-	1    9350 4450
-	1    0    0    -1
-$EndComp
-$Comp
 L power:+3.3V #PWR094
 U 1 1 5E769D6C
@@
 F 3 "~" H 8550 2700 50  0001 C CNN
 	1    8550 2700
-	1    0    0    -1
-$EndComp
-$Comp
-L power:GNDD #PWR093
-U 1 1 5E791CD6
-P 8550 2800
-F 0 "#PWR093" H 8550 2550 50  0001 C CNN
-F 1 "GNDD" H 8550 2675 50  0000 C CNN
-F 2 "" H 8550 2800 50  0001 C CNN
-F 3 "" H 8550 2800 50  0001 C CNN
-	1    8550 2800
 	1    0    0    -1
 $EndComp
@@
 $EndComp
 $Comp
-L power:GNDD #PWR091
-U 1 1 5E979D28
-P 6950 2150
-F 0 "#PWR091" H 6950 1900 50  0001 C CNN
-F 1 "GNDD" H 6950 2025 50  0000 C CNN
-F 2 "" H 6950 2150 50  0001 C CNN
-F 3 "" H 6950 2150 50  0001 C CNN
-	1    6950 2150
-	1    0    0    -1
-$EndComp
-$Comp
 L power:+3.3V #PWR090
 U 1 1 5E979D2E
@@
 F 3 "~" H 6900 3450 50  0001 C CNN
 	1    6900 3450
-	1    0    0    -1
-$EndComp
-$Comp
-L power:GNDD #PWR089
-U 1 1 5E997E69
-P 6900 3550
-F 0 "#PWR089" H 6900 3300 50  0001 C CNN
-F 1 "GNDD" H 6900 3425 50  0000 C CNN
-F 2 "" H 6900 3550 50  0001 C CNN
-F 3 "" H 6900 3550 50  0001 C CNN
-	1    6900 3550
 	1    0    0    -1
 $EndComp
@@
 	-1   0    0    1
 $EndComp
+$Comp
+L power:+3.3VADC #PWR0103
+U 1 1 5ED5582A
+P 9600 2800
+F 0 "#PWR0103" H 9750 2750 50  0001 C CNN
+F 1 "+3.3VADC" H 9600 2900 50  0000 C CNN
+F 2 "" H 9600 2800 50  0001 C CNN
+F 3 "" H 9600 2800 50  0001 C CNN
+	1    9600 2800
+	1    0    0    -1
+$EndComp
+Wire Wire Line
+	9600 2800 9450 2800
+$Comp
+L power:+3.3VADC #PWR0104
+U 1 1 5ED73AA0
+P 8600 3300
+F 0 "#PWR0104" H 8750 3250 50  0001 C CNN
+F 1 "+3.3VADC" H 8600 3400 50  0000 C CNN
+F 2 "" H 8600 3300 50  0001 C CNN
+F 3 "" H 8600 3300 50  0001 C CNN
+	1    8600 3300
+	1    0    0    -1
+$EndComp
+Wire Wire Line
+	8600 3300 8600 3350
+$Comp
+L power:+3.3VADC #PWR0105
+U 1 1 5ED91E6C
+P 6300 2050
+F 0 "#PWR0105" H 6450 2000 50  0001 C CNN
+F 1 "+3.3VADC" H 6300 2150 50  0000 C CNN
+F 2 "" H 6300 2050 50  0001 C CNN
+F 3 "" H 6300 2050 50  0001 C CNN
+	1    6300 2050
+	1    0    0    -1
+$EndComp
+$Comp
+L power:+3.3VADC #PWR0107
+U 1 1 5ED91F4D
+P 6300 3400
+F 0 "#PWR0107" H 6450 3350 50  0001 C CNN
+F 1 "+3.3VADC" H 6300 3500 50  0000 C CNN
+F 2 "" H 6300 3400 50  0001 C CNN
+F 3 "" H 6300 3400 50  0001 C CNN
+	1    6300 3400
+	1    0    0    -1
+$EndComp
+$Comp
+L power:GNDREF #PWR0108
+U 1 1 5ED923DA
+P 6600 3050
+F 0 "#PWR0108" H 6600 2800 50  0001 C CNN
+F 1 "GNDREF" H 6600 2900 50  0000 C CNN
+F 2 "" H 6600 3050 50  0001 C CNN
+F 3 "" H 6600 3050 50  0001 C CNN
+	1    6600 3050
+	1    0    0    -1
+$EndComp
+$Comp
+L power:GNDREF #PWR0109
+U 1 1 5ED93B58
+P 9050 3000
+F 0 "#PWR0109" H 9050 2750 50  0001 C CNN
+F 1 "GNDREF" H 9050 2850 50  0000 C CNN
+F 2 "" H 9050 3000 50  0001 C CNN
+F 3 "" H 9050 3000 50  0001 C CNN
+	1    9050 3000
+	1    0    0    -1
+$EndComp
+$Comp
+L power:GNDREF #PWR0110
+U 1 1 5EDB20E9
+P 7600 3200
+F 0 "#PWR0110" H 7600 2950 50  0001 C CNN
+F 1 "GNDREF" H 7600 3050 50  0000 C CNN
+F 2 "" H 7600 3200 50  0001 C CNN
+F 3 "" H 7600 3200 50  0001 C CNN
+	1    7600 3200
+	1    0    0    -1
+$EndComp
+$Comp
+L power:GNDREF #PWR0111
+U 1 1 5EDD0154
+P 7600 4550
+F 0 "#PWR0111" H 7600 4300 50  0001 C CNN
+F 1 "GNDREF" H 7600 4400 50  0000 C CNN
+F 2 "" H 7600 4550 50  0001 C CNN
+F 3 "" H 7600 4550 50  0001 C CNN
+	1    7600 4550
+	1    0    0    -1
+$EndComp
+$Comp
+L power:GNDREF #PWR0112
+U 1 1 5EDEE1BF
+P 8900 4450
+F 0 "#PWR0112" H 8900 4200 50  0001 C CNN
+F 1 "GNDREF" H 8900 4300 50  0000 C CNN
+F 2 "" H 8900 4450 50  0001 C CNN
+F 3 "" H 8900 4450 50  0001 C CNN
+	1    8900 4450
+	1    0    0    -1
+$EndComp
+$Comp
+L power:GNDREF #PWR0113
+U 1 1 5EE0C22A
+P 8600 4450
+F 0 "#PWR0113" H 8600 4200 50  0001 C CNN
+F 1 "GNDREF" H 8600 4300 50  0000 C CNN
+F 2 "" H 8600 4450 50  0001 C CNN
+F 3 "" H 8600 4450 50  0001 C CNN
+	1    8600 4450
+	1    0    0    -1
+$EndComp
+$Comp
+L power:GNDREF #PWR0114
+U 1 1 5EE2A295
+P 6300 3050
+F 0 "#PWR0114" H 6300 2800 50  0001 C CNN
+F 1 "GNDREF" H 6300 2900 50  0000 C CNN
+F 2 "" H 6300 3050 50  0001 C CNN
+F 3 "" H 6300 3050 50  0001 C CNN
+	1    6300 3050
+	1    0    0    -1
+$EndComp
+$Comp
+L power:GNDREF #PWR0115
+U 1 1 5EE48300
+P 6300 4400
+F 0 "#PWR0115" H 6300 4150 50  0001 C CNN
+F 1 "GNDREF" H 6300 4250 50  0000 C CNN
+F 2 "" H 6300 4400 50  0001 C CNN
+F 3 "" H 6300 4400 50  0001 C CNN
+	1    6300 4400
+	1    0    0    -1
+$EndComp
+$Comp
+L power:GNDREF #PWR0116
+U 1 1 5EE6636B
+P 6900 3550
+F 0 "#PWR0116" H 6900 3300 50  0001 C CNN
+F 1 "GNDREF" H 6900 3400 50  0000 C CNN
+F 2 "" H 6900 3550 50  0001 C CNN
+F 3 "" H 6900 3550 50  0001 C CNN
+	1    6900 3550
+	1    0    0    -1
+$EndComp
+$Comp
+L power:GNDREF #PWR0117
+U 1 1 5EE843D6
+P 6950 2150
+F 0 "#PWR0117" H 6950 1900 50  0001 C CNN
+F 1 "GNDREF" H 6950 2000 50  0000 C CNN
+F 2 "" H 6950 2150 50  0001 C CNN
+F 3 "" H 6950 2150 50  0001 C CNN
+	1    6950 2150
+	1    0    0    -1
+$EndComp
+$Comp
+L power:GNDREF #PWR0118
+U 1 1 5EEA2441
+P 8550 2800
+F 0 "#PWR0118" H 8550 2550 50  0001 C CNN
+F 1 "GNDREF" H 8550 2650 50  0000 C CNN
+F 2 "" H 8550 2800 50  0001 C CNN
+F 3 "" H 8550 2800 50  0001 C CNN
+	1    8550 2800
+	1    0    0    -1
+$EndComp
+$Comp
+L power:GNDREF #PWR0119
+U 1 1 5EEC134C
+P 9350 4450
+F 0 "#PWR0119" H 9350 4200 50  0001 C CNN
+F 1 "GNDREF" H 9350 4300 50  0000 C CNN
+F 2 "" H 9350 4450 50  0001 C CNN
+F 3 "" H 9350 4450 50  0001 C CNN
+	1    9350 4450
+	1    0    0    -1
+$EndComp
+$Comp
+L Device:Net-Tie_2 NT?
+U 1 1 5EEDFA05
+P 8150 5200
+F 0 "NT?" H 8150 5250 50  0000 C CNN
+F 1 "Net-Tie_2" H 8150 5150 50  0000 C CNN
+F 2 "" H 8150 5200 50  0001 C CNN
+F 3 "~" H 8150 5200 50  0001 C CNN
+	1    8150 5200
+	1    0    0    -1
+$EndComp
+$Comp
+L power:GNDREF #PWR?
+U 1 1 5EEDFB02
+P 8000 5350
+F 0 "#PWR?" H 8000 5100 50  0001 C CNN
+F 1 "GNDREF" H 8000 5200 50  0000 C CNN
+F 2 "" H 8000 5350 50  0001 C CNN
+F 3 "" H 8000 5350 50  0001 C CNN
+	1    8000 5350
+	1    0    0    -1
+$EndComp
+$Comp
+L power:GNDD #PWR?
+U 1 1 5EEDFDD1
+P 8300 5350
+F 0 "#PWR?" H 8300 5100 50  0001 C CNN
+F 1 "GNDD" H 8300 5225 50  0000 C CNN
+F 2 "" H 8300 5350 50  0001 C CNN
+F 3 "" H 8300 5350 50  0001 C CNN
+	1    8300 5350
+	1    0    0    -1
+$EndComp
+Wire Wire Line
+	8300 5350 8300 5200
+Wire Wire Line
+	8300 5200 8250 5200
+Wire Wire Line
+	8000 5350 8000 5200
+Wire Wire Line
+	8000 5200 8050 5200
 $EndSCHEMATC

Commit message: Fix INA4181 pin type
Parts:
- gave numbers to parts that had none: 1
Changed lines of the file:
@@
 	7150 3200 7300 3200
-Wire Wire Line
-	7600 3200 7600 3150
 Wire Wire Line
 	7450 3150 7450 3200
@@
 $EndComp
 $Comp
-L Device:Net-Tie_2 NT?
+L Device:Net-Tie_2 NT1
 U 1 1 5EEDFA05
 P 8150 5200
-F 0 "NT?" H 8150 5250 50  0000 C CNN
+F 0 "NT1" H 8150 5250 50  0000 C CNN
 F 1 "Net-Tie_2" H 8150 5150 50  0000 C CNN
 F 2 "" H 8150 5200 50  0001 C CNN
@@
 $EndComp
 $Comp
-L power:GNDREF #PWR?
+L power:GNDREF #PWR0120
 U 1 1 5EEDFB02
 P 8000 5350
-F 0 "#PWR?" H 8000 5100 50  0001 C CNN
+F 0 "#PWR0120" H 8000 5100 50  0001 C CNN
 F 1 "GNDREF" H 8000 5200 50  0000 C CNN
 F 2 "" H 8000 5350 50  0001 C CNN
@@
 $EndComp
 $Comp
-L power:GNDD #PWR?
+L power:GNDD #PWR0121
 U 1 1 5EEDFDD1
 P 8300 5350
-F 0 "#PWR?" H 8300 5100 50  0001 C CNN
+F 0 "#PWR0121" H 8300 5100 50  0001 C CNN
 F 1 "GNDD" H 8300 5225 50  0000 C CNN
 F 2 "" H 8300 5350 50  0001 C CNN
@@
 Wire Wire Line
 	8000 5200 8050 5200
+Connection ~ 7600 4550
+Connection ~ 7600 3200
+Wire Wire Line
+	7600 3200 7600 3150
 $EndSCHEMATC

Commit message: Add footprints
Parts:
- C17, C18, C19, C20, C21, C22, C23, C24: footprint (none) -> Capacitor_SMD:C_0805_2012Metric_Pad1.15x1.40mm_HandSolder
- C25, C30, C31: footprint (none) -> Capacitor_THT:CP_Radial_D8.0mm_P3.50mm
- M1: footprint (none) -> Connector_JST:JST_XH_B4B-XH-A_1x04_P2.50mm_Vertical
- NT1: footprint (none) -> NetTie:NetTie-2_SMD_Pad0.5mm
- R10, R3, R4, R5, R6, R7, R8, R9: footprint (none) -> Connector_JST:JST_XH_B2B-XH-A_1x02_P2.50mm_Vertical
- SW1: footprint (none) -> Connector_PinHeader_1.27mm:PinHeader_2x05_P1.27mm_Vertical
- U14: footprint (none) -> Package_SO:SOIC-16_3.9x9.9mm_P1.27mm
- U15: footprint (none) -> Package_TO_SOT_SMD:SOT-23-5_HandSoldering
Changed lines of the file:
@@
 F 0 "R3" V 5330 2250 50  0000 C CNN
 F 1 ".25m" V 5250 2250 50  0000 C CNN
-F 2 "" V 5180 2250 50  0001 C CNN
+F 2 "Connector_JST:JST_XH_B2B-XH-A_1x02_P2.50mm_Vertical" V 5180 2250 50  0001 C CNN
 F 3 "~" H 5250 2250 50  0001 C CNN
 	1    5250 2250
@@
 F 0 "R4" V 5330 2850 50  0000 C CNN
 F 1 ".25m" V 5250 2850 50  0000 C CNN
-F 2 "" V 5180 2850 50  0001 C CNN
+F 2 "Connector_JST:JST_XH_B2B-XH-A_1x02_P2.50mm_Vertical" V 5180 2850 50  0001 C CNN
 F 3 "~" H 5250 2850 50  0001 C CNN
 	1    5250 2850
@@
 F 0 "R5" V 5330 3450 50  0000 C CNN
 F 1 ".25m" V 5250 3450 50  0000 C CNN
-F 2 "" V 5180 3450 50  0001 C CNN
+F 2 "Connector_JST:JST_XH_B2B-XH-A_1x02_P2.50mm_Vertical" V 5180 3450 50  0001 C CNN
 F 3 "~" H 5250 3450 50  0001 C CNN
 	1    5250 3450
@@
 F 0 "R6" V 5330 4050 50  0000 C CNN
 F 1 ".25m" V 5250 4050 50  0000 C CNN
-F 2 "" V 5180 4050 50  0001 C CNN
+F 2 "Connector_JST:JST_XH_B2B-XH-A_1x02_P2.50mm_Vertical" V 5180 4050 50  0001 C CNN
 F 3 "~" H 5250 4050 50  0001 C CNN
 	1    5250 4050
@@
 F 0 "R7" V 5330 4650 50  0000 C CNN
 F 1 ".25m" V 5250 4650 50  0000 C CNN
-F 2 "" V 5180 4650 50  0001 C CNN
+F 2 "Connector_JST:JST_XH_B2B-XH-A_1x02_P2.50mm_Vertical" V 5180 4650 50  0001 C CNN
 F 3 "~" H 5250 4650 50  0001 C CNN
 	1    5250 4650
@@
 F 0 "U15" H 9300 3050 50  0000 C CNN
 F 1 "REF2033" H 9200 2950 50  0000 C CNN
-F 2 "" H 9200 2700 50  0001 C CNN
+F 2 "Package_TO_SOT_SMD:SOT-23-5_HandSoldering" H 9200 2700 50  0001 C CNN
 F 3 "http://www.ti.com/lit/ds/symlink/ref2033.pdf" H 9200 2700 50  0001 C CNN
 	1    9100 2700
@@
 F 0 "R8" V 5330 5250 50  0000 C CNN
 F 1 ".25m" V 5250 5250 50  0000 C CNN
-F 2 "" V 5180 5250 50  0001 C CNN
+F 2 "Connector_JST:JST_XH_B2B-XH-A_1x02_P2.50mm_Vertical" V 5180 5250 50  0001 C CNN
 F 3 "~" H 5250 5250 50  0001 C CNN
 	1    5250 5250
@@
 F 0 "R9" V 5330 5850 50  0000 C CNN
 F 1 ".25m" V 5250 5850 50  0000 C CNN
-F 2 "" V 5180 5850 50  0001 C CNN
+F 2 "Connector_JST:JST_XH_B2B-XH-A_1x02_P2.50mm_Vertical" V 5180 5850 50  0001 C CNN
 F 3 "~" H 5250 5850 50  0001 C CNN
 	1    5250 5850
@@
 F 0 "R10" V 5330 6450 50  0000 C CNN
 F 1 ".25m" V 5250 6450 50  0000 C CNN
-F 2 "" V 5180 6450 50  0001 C CNN
+F 2 "Connector_JST:JST_XH_B2B-XH-A_1x02_P2.50mm_Vertical" V 5180 6450 50  0001 C CNN
 F 3 "~" H 5250 6450 50  0001 C CNN
 	1    5250 6450
@@
 F 0 "U14" H 9150 4400 50  0000 C CNN
 F 1 "MCP3008" H 9100 4300 50  0000 C CNN
-F 2 "" H 8800 3950 50  0001 C CNN
+F 2 "Package_SO:SOIC-16_3.9x9.9mm_P1.27mm" H 8800 3950 50  0001 C CNN
 F 3 "http://ww1.microchip.com/downloads/en/DeviceDoc/21295d.pdf" H 8800 3950 50  0001 C CNN
 	1    8700 3850
@@
 F 0 "SW1" H 6150 5300 50  0000 C CNN
 F 1 "SRX_Encoder" H 6050 5200 50  0000 C CNN
-F 2 "" H 5875 4810 50  0001 C CNN
+F 2 "Connector_PinHeader_1.27mm:PinHeader_2x05_P1.27mm_Vertical" H 5875 4810 50  0001 C CNN
 F 3 "~" H 5725 4910 50  0001 C CNN
 	1    6100 4900
@@
 F 0 "C24" H 7610 4470 50  0000 L CNN
 F 1 "10n" H 7610 4320 50  0000 L CNN
-F 2 "" H 7600 4400 50  0001 C CNN
+F 2 "Capacitor_SMD:C_0805_2012Metric_Pad1.15x1.40mm_HandSolder" H 7600 4400 50  0001 C CNN
 F 3 "~" H 7600 4400 50  0001 C CNN
 	1    7600 4400
@@
 F 0 "C22" H 7460 4470 50  0000 L CNN
 F 1 "10n" H 7460 4320 50  0000 L CNN
-F 2 "" H 7450 4400 50  0001 C CNN
+F 2 "Capacitor_SMD:C_0805_2012Metric_Pad1.15x1.40mm_HandSolder" H 7450 4400 50  0001 C CNN
 F 3 "~" H 7450 4400 50  0001 C CNN
 	1    7450 4400
@@
 F 0 "C20" H 7310 4470 50  0000 L CNN
 F 1 "10n" H 7310 4320 50  0000 L CNN
-F 2 "" H 7300 4400 50  0001 C CNN
+F 2 "Capacitor_SMD:C_0805_2012Metric_Pad1.15x1.40mm_HandSolder" H 7300 4400 50  0001 C CNN
 F 3 "~" H 7300 4400 50  0001 C CNN
 	1    7300 4400
@@
 F 0 "C18" H 7160 4470 50  0000 L CNN
 F 1 "10n" H 7160 4320 50  0000 L CNN
-F 2 "" H 7150 4400 50  0001 C CNN
+F 2 "Capacitor_SMD:C_0805_2012Metric_Pad1.15x1.40mm_HandSolder" H 7150 4400 50  0001 C CNN
 F 3 "~" H 7150 4400 50  0001 C CNN
 	1    7150 4400
@@
 F 0 "C23" H 7610 3120 50  0000 L CNN
 F 1 "10n" H 7610 2970 50  0000 L CNN
-F 2 "" H 7600 3050 50  0001 C CNN
+F 2 "Capacitor_SMD:C_0805_2012Metric_Pad1.15x1.40mm_HandSolder" H 7600 3050 50  0001 C CNN
 F 3 "~" H 7600 3050 50  0001 C CNN
 	1    7600 3050
@@
 F 0 "C21" H 7460 3120 50  0000 L CNN
 F 1 "10n" H 7460 2970 50  0000 L CNN
-F 2 "" H 7450 3050 50  0001 C CNN
+F 2 "Capacitor_SMD:C_0805_2012Metric_Pad1.15x1.40mm_HandSolder" H 7450 3050 50  0001 C CNN
 F 3 "~" H 7450 3050 50  0001 C CNN
 	1    7450 3050
@@
 F 0 "C19" H 7310 3120 50  0000 L CNN
 F 1 "10n" H 7310 2970 50  0000 L CNN
-F 2 "" H 7300 3050 50  0001 C CNN
+F 2 "Capacitor_SMD:C_0805_2012Metric_Pad1.15x1.40mm_HandSolder" H 7300 3050 50  0001 C CNN
 F 3 "~" H 7300 3050 50  0001 C CNN
 	1    7300 3050
@@
 F 0 "C17" H 7160 3120 50  0000 L CNN
 F 1 "10n" H 7160 2970 50  0000 L CNN
-F 2 "" H 7150 3050 50  0001 C CNN
+F 2 "Capacitor_SMD:C_0805_2012Metric_Pad1.15x1.40mm_HandSolder" H 7150 3050 50  0001 C CNN
 F 3 "~" H 7150 3050 50  0001 C CNN
 	1    7150 3050
@@
 F 0 "M1" H 5000 7475 50  0000 L CNN
 F 1 "Hopper_Servo" H 5000 7100 50  0000 L TNN
-F 2 "" H 5200 7110 50  0001 C CNN
+F 2 "Connector_JST:JST_XH_B4B-XH-A_1x04_P2.50mm_Vertical" H 5200 7110 50  0001 C CNN
 F 3 "http://forums.parallax.com/uploads/attachments/46831/74481.png" H 5200 7110 50  0001 C CNN
 	1    5200 7300
@@
 F 0 "C25" H 4625 7450 50  0000 L CNN
 F 1 "470u" H 4625 7250 50  0000 L CNN
-F 2 "" H 4638 7200 50  0001 C CNN
+F 2 "Capacitor_THT:CP_Radial_D8.0mm_P3.50mm" H 4638 7200 50  0001 C CNN
 F 3 "~" H 4600 7350 50  0001 C CNN
 	1    4600 7350
@@
 F 0 "C31" H 10025 3350 50  0000 L CNN
 F 1 "470u" H 10025 3150 50  0000 L CNN
-F 2 "" H 10038 3100 50  0001 C CNN
+F 2 "Capacitor_THT:CP_Radial_D8.0mm_P3.50mm" H 10038 3100 50  0001 C CNN
 F 3 "~" H 10000 3250 50  0001 C CNN
 	1    10000 3250
@@
 F 0 "C30" H 9975 2650 50  0000 L CNN
 F 1 "470u" H 9975 2450 50  0000 L CNN
-F 2 "" H 9988 2400 50  0001 C CNN
+F 2 "Capacitor_THT:CP_Radial_D8.0mm_P3.50mm" H 9988 2400 50  0001 C CNN
 F 3 "~" H 9950 2550 50  0001 C CNN
 	1    9950 2550
@@
 F 0 "NT1" H 8150 5250 50  0000 C CNN
 F 1 "Net-Tie_2" H 8150 5150 50  0000 C CNN
-F 2 "" H 8150 5200 50  0001 C CNN
+F 2 "NetTie:NetTie-2_SMD_Pad0.5mm" H 8150 5200 50  0001 C CNN
 F 3 "~" H 8150 5200 50  0001 C CNN
 	1    8150 5200

Commit message: Change big cap footprint
Parts:
- C3: footprint Capacitor_THT:CP_Radial_D10.0mm_P2.50mm -> Capacitor_THT:CP_Radial_D8.0mm_P3.50mm
Changed lines of the file:
@@
 F 0 "C3" H 8068 996 50  0000 L CNN
 F 1 "1000uF" H 8068 905 50  0000 L CNN
-F 2 "Capacitor_THT:CP_Radial_D10.0mm_P2.50mm" H 7988 800 50  0001 C CNN
+F 2 "Capacitor_THT:CP_Radial_D8.0mm_P3.50mm" H 7988 800 50  0001 C CNN
 F 3 "~" H 7950 950 50  0001 C CNN
 	1    7950 950
@@
 	1    0    0    -1
 $EndComp
-Connection ~ 8050 2600
 NoConn ~ 2700 5000
 NoConn ~ 6450 5100
@@
 Wire Wire Line
 	7600 3200 7600 3150
+Connection ~ 8050 2600
 $EndSCHEMATC
