File: kicad-eboard/kicad-eboard.sch (KiCad schematic (older format))
At the start: 81 parts, among them J1 Conn_01x02, J2 Conn_02x03, M1 Hopper_Servo, SW1 SRX_Encoder, SW4 LIMIT_1, SW5 LIMIT_2, U1 TinkerBoard, U10 Sabertooth2x60, U11 Sabertooth2x60, U12 Sabertooth2x60, U13 INA4181, U14 MCP3008, U15 REF2033, U2 ADS1015IDGS, U3 INA4181, U4 Hokuyo_UST-10LX, U5 Hokuyo_UST-10LX, U6 PDQ15-Q24-S12-D, U7 PDQ30-Q24-S5-D, U8 Sabertooth2x60

Commit message: Add capacitor array symbol
Parts:
- removed C17, C18, C19, C20, C21, C22, C23, C24: 10n, Capacitor_SMD:C_0805_2012Metric_Pad1.15x1.40mm_HandSolder, symbol Device:C_Small
- added C17, C32: 10n, symbol 2019Spacehawks:C_Pack04_Split
Connections:
- wire segments 324 -> 327
Changed lines of the file:
@@
 Wire Wire Line
 	8050 3550 8100 3550
-$Comp
-L Device:C_Small C24
-U 1 1 602A3F86
-P 7600 4400
-F 0 "C24" H 7610 4470 50  0000 L CNN
-F 1 "10n" H 7610 4320 50  0000 L CNN
-F 2 "Capacitor_SMD:C_0805_2012Metric_Pad1.15x1.40mm_HandSolder" H 7600 4400 50  0001 C CNN
-F 3 "~" H 7600 4400 50  0001 C CNN
-	1    7600 4400
-	1    0    0    -1
-$EndComp
-$Comp
-L Device:C_Small C22
-U 1 1 602A4119
-P 7450 4400
-F 0 "C22" H 7460 4470 50  0000 L CNN
-F 1 "10n" H 7460 4320 50  0000 L CNN
-F 2 "Capacitor_SMD:C_0805_2012Metric_Pad1.15x1.40mm_HandSolder" H 7450 4400 50  0001 C CNN
-F 3 "~" H 7450 4400 50  0001 C CNN
-	1    7450 4400
-	1    0    0    -1
-$EndComp
-$Comp
-L Device:C_Small C20
-U 1 1 602A411F
-P 7300 4400
-F 0 "C20" H 7310 4470 50  0000 L CNN
-F 1 "10n" H 7310 4320 50  0000 L CNN
-F 2 "Capacitor_SMD:C_0805_2012Metric_Pad1.15x1.40mm_HandSolder" H 7300 4400 50  0001 C CNN
-F 3 "~" H 7300 4400 50  0001 C CNN
-	1    7300 4400
-	1    0    0    -1
-$EndComp
-$Comp
-L Device:C_Small C18
-U 1 1 602F9A32
-P 7150 4400
-F 0 "C18" H 7160 4470 50  0000 L CNN
-F 1 "10n" H 7160 4320 50  0000 L CNN
-F 2 "Capacitor_SMD:C_0805_2012Metric_Pad1.15x1.40mm_HandSolder" H 7150 4400 50  0001 C CNN
-F 3 "~" H 7150 4400 50  0001 C CNN
-	1    7150 4400
-	1    0    0    -1
-$EndComp
 Wire Wire Line
 	7450 4300 7450 4150
@@
 Wire Wire Line
 	7300 4550 7450 4550
-$Comp
-L Device:C_Small C23
-U 1 1 60653C4F
-P 7600 3050
-F 0 "C23" H 7610 3120 50  0000 L CNN
-F 1 "10n" H 7610 2970 50  0000 L CNN
-F 2 "Capacitor_SMD:C_0805_2012Metric_Pad1.15x1.40mm_HandSolder" H 7600 3050 50  0001 C CNN
-F 3 "~" H 7600 3050 50  0001 C CNN
-	1    7600 3050
-	1    0    0    -1
-$EndComp
-$Comp
-L Device:C_Small C21
-U 1 1 60653C55
-P 7450 3050
-F 0 "C21" H 7460 3120 50  0000 L CNN
-F 1 "10n" H 7460 2970 50  0000 L CNN
-F 2 "Capacitor_SMD:C_0805_2012Metric_Pad1.15x1.40mm_HandSolder" H 7450 3050 50  0001 C CNN
-F 3 "~" H 7450 3050 50  0001 C CNN
-	1    7450 3050
-	1    0    0    -1
-$EndComp
-$Comp
-L Device:C_Small C19
-U 1 1 60653C5B
-P 7300 3050
-F 0 "C19" H 7310 3120 50  0000 L CNN
-F 1 "10n" H 7310 2970 50  0000 L CNN
-F 2 "Capacitor_SMD:C_0805_2012Metric_Pad1.15x1.40mm_HandSolder" H 7300 3050 50  0001 C CNN
-F 3 "~" H 7300 3050 50  0001 C CNN
-	1    7300 3050
-	1    0    0    -1
-$EndComp
-$Comp
-L Device:C_Small C17
-U 1 1 60653C61
-P 7150 3050
-F 0 "C17" H 7160 3120 50  0000 L CNN
-F 1 "10n" H 7160 2970 50  0000 L CNN
-F 2 "Capacitor_SMD:C_0805_2012Metric_Pad1.15x1.40mm_HandSolder" H 7150 3050 50  0001 C CNN
-F 3 "~" H 7150 3050 50  0001 C CNN
-	1    7150 3050
-	1    0    0    -1
-$EndComp
-Wire Wire Line
-	7450 2950 7450 2800
 Wire Wire Line
 	7450 2800 7100 2800
-Wire Wire Line
-	7300 2950 7300 2700
-Wire Wire Line
-	7150 2950 7150 2600
 $Comp
 L Device:R_Pack04_Split R11
@@
 	7100 2700 7300 2700
 Wire Wire Line
-	7100 2900 7600 2900
+	7100 2900 7150 2900
 Wire Wire Line
 	7600 2950 7600 2900
@@
 	7600 3200 7600 3150
 Connection ~ 8050 2600
+$Comp
+L 2019Spacehawks:C_Pack04_Split C32
+U 1 1 5F09CA3E
+P 7150 3050
+F 0 "C32" H 7160 3120 50  0000 L CNN
+F 1 "10n" H 7160 2970 50  0000 L CNN
+F 2 "" H 7150 3050 50  0001 C CNN
+F 3 "~" H 7150 3050 50  0001 C CNN
+	1    7150 3050
+	1    0    0    -1
+$EndComp
+$Comp
+L 2019Spacehawks:C_Pack04_Split C32
+U 2 1 5F09CF4D
+P 7300 3050
+F 0 "C32" H 7310 3120 50  0001 L CNN
+F 1 "10n" H 7310 2970 50  0000 L CNN
+F 2 "" H 7300 3050 50  0001 C CNN
+F 3 "~" H 7300 3050 50  0001 C CNN
+	2    7300 3050
+	1    0    0    -1
+$EndComp
+$Comp
+L 2019Spacehawks:C_Pack04_Split C32
+U 3 1 5F157B86
+P 7450 3050
+F 0 "C32" H 7460 3120 50  0001 L CNN
+F 1 "10n" H 7460 2970 50  0000 L CNN
+F 2 "" H 7450 3050 50  0001 C CNN
+F 3 "~" H 7450 3050 50  0001 C CNN
+	3    7450 3050
+	1    0    0    -1
+$EndComp
+$Comp
+L 2019Spacehawks:C_Pack04_Split C32
+U 4 1 5F157E9C
+P 7600 3050
+F 0 "C32" H 7610 3120 50  0001 L CNN
+F 1 "10n" H 7610 2970 50  0000 L CNN
+F 2 "" H 7600 3050 50  0001 C CNN
+F 3 "~" H 7600 3050 50  0001 C CNN
+	4    7600 3050
+	1    0    0    -1
+$EndComp
+Wire Wire Line
+	7150 2900 7300 2900
+Wire Wire Line
+	7300 2900 7450 2900
+Wire Wire Line
+	7450 2900 7600 2900
+Wire Wire Line
+	7150 2600 7150 2950
+Wire Wire Line
+	7300 2700 7300 2950
+Wire Wire Line
+	7450 2800 7450 2950
+$Comp
+L 2019Spacehawks:C_Pack04_Split C17
+U 1 1 5F23490B
+P 7150 4400
+F 0 "C17" H 7160 4470 50  0000 L CNN
+F 1 "10n" H 7160 4320 50  0000 L CNN
+F 2 "" H 7150 4400 50  0001 C CNN
+F 3 "~" H 7150 4400 50  0001 C CNN
+	1    7150 4400
+	1    0    0    -1
+$EndComp
+$Comp
+L 2019Spacehawks:C_Pack04_Split C17
+U 2 1 5F234911
+P 7300 4400
+F 0 "C17" H 7310 4470 50  0001 L CNN
+F 1 "10n" H 7310 4320 50  0000 L CNN
+F 2 "" H 7300 4400 50  0001 C CNN
+F 3 "~" H 7300 4400 50  0001 C CNN
+	2    7300 4400
+	1    0    0    -1
+$EndComp
+$Comp
+L 2019Spacehawks:C_Pack04_Split C17
+U 3 1 5F234917
+P 7450 4400
+F 0 "C17" H 7460 4470 50  0001 L CNN
+F 1 "10n" H 7460 4320 50  0000 L CNN
+F 2 "" H 7450 4400 50  0001 C CNN
+F 3 "~" H 7450 4400 50  0001 C CNN
+	3    7450 4400
+	1    0    0    -1
+$EndComp
+$Comp
+L 2019Spacehawks:C_Pack04_Split C17
+U 4 1 5F23491D
+P 7600 4400
+F 0 "C17" H 7610 4470 50  0001 L CNN
+F 1 "10n" H 7610 4320 50  0000 L CNN
+F 2 "" H 7600 4400 50  0001 C CNN
+F 3 "~" H 7600 4400 50  0001 C CNN
+	4    7600 4400
+	1    0    0    -1
+$EndComp
 $EndSCHEMATC

Commit message: Add capacitor array footprint
Parts:
- removed C17: 10n, symbol 2019Spacehawks:C_Pack04_Split
- removed unit 2 of C32
- removed unit 3 of C32
- removed unit 4 of C32
- added unit 2 of C6
- added unit 3 of C6
- added unit 4 of C6
- added C7: 10n, 2019Spacehawks:C_Array_Convex_4x0612, symbol 2019Spacehawks:C_Pack04_Split
- C6: renamed from C32; footprint (none) -> 2019Spacehawks:C_Array_Convex_4x0612
- renumbered C28 to C10, C5 to C11, C6 to C12, C7 to C13, C8 to C14, C9 to C15, C10 to C16, C29 to C17, C30 to C18, C31 to C19, C4 to C20, C15 to C21, C25 to C3, C26 to C4, C27 to C5, C16 to C8, C3 to C9, J2 to J1, J1 to J2, R3 to R1, R12 to R10, R36 to R11, R4 to R2, R5 to R3, R6 to R4, R7 to R5, R8 to R6, R9 to R7, R10 to R8, R11 to R9, RV3 to RV1, RV4 to RV2, RV5 to RV3, RV1 to RV4, RV2 to RV5, SW4 to SW1, SW5 to SW2, SW1 to SW3, TP3 to TP1, TP15 to TP10, TP6 to TP11, TP9 to TP12, TP7 to TP13, TP10 to TP14, TP8 to TP15, TP11 to TP2, TP12 to TP3, TP13 to TP4, TP1 to TP5, TP2 to TP6, TP14 to TP7, TP5 to TP8, TP4 to TP9, U15 to U10, U6 to U11, U7 to U12, U4 to U13, U5 to U14, U8 to U2, U10 to U3, U11 to U4, U12 to U5, U3 to U6, U13 to U7, U2 to U8, U14 to U9
