File: kicad-eboard/I2CtoPWM.sch (KiCad schematic (older format))
At the start: 61 parts, among them Q1 AOD417

Commit message: Satisfy some ERC things
Parts:
- gave numbers to parts that had none: 46
- renumbered C1 to C3, C2 to C4, SJ_A0 to SJ_A1, SJ_A1 to SJ_A2, SJ_A2 to SJ_A3, SJ_A3 to SJ_A4, SJ_A4 to SJ_A5, SJ_A5 to SJ_A6

Commit message: Use serial instead of analog Sabertooth ctrl
Changed lines of the file:
@@
 $EndComp
-Wire Wire Line
-	3900 6500 3950 6500
-Wire Wire Line
-	3950 6600 3900 6600
 Wire Wire Line
 	3950 6800 4250 6800
@@
 Text HLabel 2250 6900 2    50   Input ~ 0
 GND
+Wire Wire Line
+	3950 6600 3900 6600
+Wire Wire Line
+	3950 6500 3900 6500
 Wire Bus Line
 	6400 1950 6400 3700
+$Comp
+L power:PWR_FLAG #FLG0107
+U 1 1 5E0815A6
+P 3950 6300
+F 0 "#FLG0107" H 3950 6375 50  0001 C CNN
+F 1 "PWR_FLAG" H 3950 6450 50  0000 C CNN
+F 2 "" H 3950 6300 50  0001 C CNN
+F 3 "~" H 3950 6300 50  0001 C CNN
+	1    3950 6300
+	1    0    0    -1
+$EndComp
+Connection ~ 3950 6300
 $EndSCHEMATC
