File: kicad-eboard/MP6050.sch (KiCad schematic (older format))
At the start: 11 parts, among them J19 Conn_01x10, U9 MPU-6050

Commit message: Add some footprints
Parts:
- C11, C12, C13, C14: footprint (none) -> Capacitor_SMD:C_0805_2012Metric_Pad1.15x1.40mm_HandSolder
- J19: value Conn_01x10 -> #Conn_01x10
- JP1: footprint (none) -> Jumper:SolderJumper-3_P1.3mm_Bridged12_RoundedPad1.0x1.5mm_NumberLabels
- JP2, JP3: footprint (none) -> Jumper:SolderJumper-2_P1.3mm_Bridged_RoundedPad1.0x1.5mm
- R1, R2: footprint (none) -> Resistor_SMD:R_0603_1608Metric_Pad1.05x0.95mm_HandSolder
Changed lines of the file:
@@
 F 0 "C14" H 6810 5715 59  0000 L BNN
 F 1 "2.2nF" H 6810 5515 59  0000 L BNN
-F 2 "" H 6750 5600 50  0001 C CNN
+F 2 "Capacitor_SMD:C_0805_2012Metric_Pad1.15x1.40mm_HandSolder" H 6750 5600 50  0001 C CNN
 F 3 "" H 6750 5600 50  0001 C CNN
 	1    6750 5600
@@
 F 0 "C13" H 6360 4115 59  0000 L BNN
 F 1 "0.1uF" H 6360 3915 59  0000 L BNN
-F 2 "" H 6300 4000 50  0001 C CNN
+F 2 "Capacitor_SMD:C_0805_2012Metric_Pad1.15x1.40mm_HandSolder" H 6300 4000 50  0001 C CNN
 F 3 "" H 6300 4000 50  0001 C CNN
 	1    6300 4000
@@
 F 0 "C11" H 5160 4015 59  0000 L BNN
 F 1 "10nF" H 5160 3815 59  0000 L BNN
-F 2 "" H 5100 3900 50  0001 C CNN
+F 2 "Capacitor_SMD:C_0805_2012Metric_Pad1.15x1.40mm_HandSolder" H 5100 3900 50  0001 C CNN
 F 3 "" H 5100 3900 50  0001 C CNN
 	1    5100 3900
@@
 F 0 "JP2" H 4400 6080 50  0000 C CNN
 F 1 "SolderJumper_2_Bridged" H 4400 5900 50  0000 C CNN
-F 2 "" H 4400 6000 50  0001 C CNN
+F 2 "Jumper:SolderJumper-2_P1.3mm_Bridged_RoundedPad1.0x1.5mm" H 4400 6000 50  0001 C CNN
 F 3 "~" H 4400 6000 50  0001 C CNN
 	1    4400 6000
@@
 F 0 "JP3" H 4700 6080 50  0000 C CNN
 F 1 "SolderJumper_2_Bridged" H 4700 5900 50  0000 C CNN
-F 2 "" H 4700 6000 50  0001 C CNN
+F 2 "Jumper:SolderJumper-2_P1.3mm_Bridged_RoundedPad1.0x1.5mm" H 4700 6000 50  0001 C CNN
 F 3 "~" H 4700 6000 50  0001 C CNN
 	1    4700 6000
@@
 F 0 "JP1" H 3850 4900 50  0000 C CNN
 F 1 "SolderJumper_3_Bridged12" H 3950 5110 50  0000 C CNN
-F 2 "" H 3950 5000 50  0001 C CNN
+F 2 "Jumper:SolderJumper-3_P1.3mm_Bridged12_RoundedPad1.0x1.5mm_NumberLabels" H 3950 5000 50  0001 C CNN
 F 3 "~" H 3950 5000 50  0001 C CNN
 	1    3950 5000
@@
 AR Path="/5DCD5C02/5DAEBC3C" Ref="J?"  Part="1"
 F 0 "J19" H 1700 4800 50  0000 C CNN
-F 1 "Conn_01x10" H 1700 3700 50  0000 C CNN
+F 1 "#Conn_01x10" H 1700 3700 50  0000 C CNN
 F 2 "" H 1700 4300 50  0001 C CNN
 F 3 "~" H 1700 4300 50  0001 C CNN
@@
 F 0 "R1" V 4430 4300 50  0000 C CNN
 F 1 "10K" V 4350 4300 50  0000 C CNN
-F 2 "" V 4280 4300 50  0001 C CNN
+F 2 "Resistor_SMD:R_0603_1608Metric_Pad1.05x0.95mm_HandSolder" V 4280 4300 50  0001 C CNN
 F 3 "~" H 4350 4300 50  0001 C CNN
 	1    4350 4300
@@
 F 0 "R2" V 4680 4100 50  0000 C CNN
 F 1 "10K" V 4600 4100 50  0000 C CNN
-F 2 "" V 4530 4100 50  0001 C CNN
+F 2 "Resistor_SMD:R_0603_1608Metric_Pad1.05x0.95mm_HandSolder" V 4530 4100 50  0001 C CNN
 F 3 "~" H 4600 4100 50  0001 C CNN
 	1    4600 4100
@@
 F 0 "C12" H 6260 5865 59  0000 L BNN
 F 1 "0.1uF" H 6260 5665 59  0000 L BNN
-F 2 "" H 6200 5750 50  0001 C CNN
+F 2 "Capacitor_SMD:C_0805_2012Metric_Pad1.15x1.40mm_HandSolder" H 6200 5750 50  0001 C CNN
 F 3 "" H 6200 5750 50  0001 C CNN
 	1    6200 5750

Commit message: Move #s to actually work
Parts:
- removed J19: #Conn_01x10, symbol Connector_Generic:Conn_01x10
Connections:
- net labels added: Conn_01x10
Changed lines of the file:
@@
 ***
 $Comp
-L Connector_Generic:Conn_01x10 J19
+L Connector_Generic:Conn_01x10 #J19
 U 1 1 5DAEBC3C
 P 1700 4300
-AR Path="/5DAF980D/5DAEBC3C" Ref="J19"  Part="1"
+AR Path="/5DAF980D/5DAEBC3C" Ref="#J19"  Part="1"
 AR Path="/5DCD5C02/5DAEBC3C" Ref="J?"  Part="1"
-F 0 "J19" H 1700 4800 50  0000 C CNN
-F 1 "#Conn_01x10" H 1700 3700 50  0000 C CNN
+F 0 "#J19" H 1700 4800 50  0000 C CNN
+F 1 "Conn_01x10" H 1700 3700 50  0000 C CNN
 F 2 "" H 1700 4300 50  0001 C CNN
 F 3 "~" H 1700 4300 50  0001 C CNN

Commit message: Scratch
Parts:
- added J19: Conn_01x10, Connector_PinHeader_2.54mm:PinHeader_1x10_P2.54mm_Vertical, symbol Connector_Generic:Conn_01x10
Connections:
- net labels removed: Conn_01x10
Changed lines of the file:
@@
 ***
 $Comp
-L Connector_Generic:Conn_01x10 #J19
+L Connector_Generic:Conn_01x10 J19
 U 1 1 5DAEBC3C
 P 1700 4300
-AR Path="/5DAF980D/5DAEBC3C" Ref="#J19"  Part="1"
+AR Path="/5DAF980D/5DAEBC3C" Ref="J19"  Part="1"
 AR Path="/5DCD5C02/5DAEBC3C" Ref="J?"  Part="1"
-F 0 "#J19" H 1700 4800 50  0000 C CNN
+F 0 "J19" H 1700 4800 50  0000 C CNN
 F 1 "Conn_01x10" H 1700 3700 50  0000 C CNN
-F 2 "" H 1700 4300 50  0001 C CNN
+F 2 "Connector_PinHeader_2.54mm:PinHeader_1x10_P2.54mm_Vertical" H 1700 4300 50  0001 C CNN
 F 3 "~" H 1700 4300 50  0001 C CNN
 	1    1700 4300
